Commit message: Update test.urdf

File: urdf/test.urdf (robot description, URDF)
Before this commit: robot belaaaaaaaaaaaaaaaaaaaaaaazik, 5 links, 4 joints
Links:
- added link odom
Joints:
- removed joint joint_front_left
- removed joint joint_rear_left
- removed joint joint_rear_right
- added joint odom_to_base: type fixed, parent odom, child base_link
- added joint rack_pinion_joint: type revolute, parent base_link, child wheel_front_left, origin xyz=0.4 0.25 0.1 rpy=0 0 0, axis 0 0 1, limit lower=-1.57 upper=1.57 effort=10.0 velocity=1.0
- added joint wheel_rear_left: type continuous, parent base_link, child wheel_rear_left, origin xyz=-0.4 0.25 0.1, axis 0 0 1
- added joint wheel_rear_right: type continuous, parent base_link, child wheel_rear_right, origin xyz=-0.4 -0.25 0.1, axis 0 0 1
- joint joint_front_right: origin xyz=0.4 -0.25 0.1 -> xyz=0.4 -0.25 0.1 rpy=0 0 0
